File: emb/adc/adc.brd (EAGLE design)
At the start: 100 x 80 mm, 21 parts, among them IC1 AD623N, IC2 MCP3008, Q1 RD06HVF1, Q2 RD06HVF1, Q3 RD06HVF1, Q4 RD06HVF1

Commit message: new board
Parts:
- removed LED_YELLOW: (no value), adafruit:LED5MM
- removed Q4: RD06HVF1, transistor-power:RD06HVF1
- added R10, R9: 12K, rcl:0207/10
- IC1: value AD623N -> LM358N; device analog-devices:DIL08 -> linear:DIL08
- Q1, Q2, Q3: value RD06HVF1 -> (none); device transistor-power:RD06HVF1 -> adafruit:TO220V
- R1: value (none) -> 100K
- R2: value (none) -> 7.5K
- R3: value (none) -> 1.2K
- R4: value (none) -> 3.3K
- R5: value (none) -> 200
- R6, R7: value (none) -> 160
- R8: value (none) -> 12K
- moved R8 74.8 mm to (75.0, 58.0), turned to 0 degrees
- moved R7 48.5 mm to (59.2, 39.5), turned to 270 degrees
- moved R5 32.2 mm to (40.3, 48.4), turned to 225 degrees
- moved R2 22.9 mm to (34.7, 36.5), turned to 180 degrees
- moved R6 19.7 mm to (34.7, 39.3)
- moved J2 18.0 mm to (71.0, 37.0)
- moved Q3 16.1 mm to (61.3, 51.1), turned to 270 degrees
- moved LED_GREEN 15.9 mm to (43.0, 43.3), turned to 0 degrees
- moved Q1 15.8 mm to (72.8, 51.1), turned to 270 degrees
- moved Q2 15.7 mm to (67.2, 50.9), turned to 270 degrees
- moved R3 14.1 mm to (26.3, 58.7), turned to 270 degrees
- moved R1 13.7 mm to (33.5, 52.6), turned to 135 degrees
- moved LED_BLUE 11.2 mm to (54.0, 43.3), turned to 180 degrees
- moved IC2 9.59 mm to (46.0, 59.0)
- moved LED_RED 9.15 mm to (48.1, 49.6), turned to 270 degrees
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Connections:
- net N$12 renamed 3.3V
- removed net -V: IC1.4
- removed net L_Y: J1.4, Q4.1
- removed net N$14: LED_RED.A, Q1.3
- removed net N$16: LED_GREEN.K, R6.1
- removed net N$17: LED_GREEN.A, Q2.3
- removed net N$18: LED_BLUE.K, R7.1
- removed net N$19: LED_YELLOW.K, R8.1
- removed net N$20: LED_BLUE.A, Q3.3
- removed net N$21: LED_YELLOW.A, Q4.3
- removed net VCC: IC2.9
- new net 4.5V: IC1.8, R2.2, R3.2
- new net N$12: LED_GREEN.A, R6.1
- new net N$8: LED_BLUE.A, R7.1
- net 0V: now also D1.A, IC1.4, IC2.9, Q1.3, Q2.3, Q3.3, R10.1, R4.2, R8.2, R9.2; no longer IC1.5, Q1.2, Q2.2, Q3.2, Q4.2, R3.2
- net 12V: now also R2.1; no longer D1.A, IC1.7, R4.2, R8.2
- net L_B: now also R10.2
- net L_G: now also R9.1
- net L_R: now also R8.1
- net N$1: now also D1.K, IC1.3; no longer IC1.1
- net N$13: now also LED_GREEN.K, Q2.2; no longer LED_RED.K, R5.1
- net N$2: now also LED_BLUE.K, Q3.2; no longer IC1.8, R1.1
- net N$3: now also LED_RED.A, R5.1; no longer D1.K, R2.1
- net N$6: now also LED_RED.K, Q1.2; no longer IC1.3, R2.2
- net N$7: now also IC1.1, R1.1; no longer IC1.6
Routing:
- net L_G: track 354.1 -> 19.2 mm
- net 0V: track 170.6 -> 0.00 mm
- net 12V: track 219.9 -> 60.1 mm
- net L_Y: track 101.4 -> 0.00 mm
- net L_B: track 86.5 -> 16.5 mm
- net L_R: track 82.9 -> 19.1 mm
- net N$18: track 54.5 -> 0.00 mm
- net N$7: track 69.0 -> 16.0 mm
- net N$1: track 6.35 -> 55.9 mm
- net N$19: track 47.1 -> 0.00 mm
- net N$16: track 43.7 -> 0.00 mm
- net N$6: track 14.7 -> 56.8 mm
- net N$13: track 69.1 -> 29.7 mm
- net N$20: track 34.1 -> 0.00 mm
- net N$17: track 28.9 -> 0.00 mm
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- added copper zone on layer 1, net 0V
Other:
- board size 100 x 80 mm -> 99.5 x 79.8 mm
- board text added: "LED_BOARD"

Commit message: adc files updated
Parts:
- added J3: (no value), con-amp:10X02MTA
- moved R2 3.24 mm to (36.8, 34.0)
- moved R5 2.16 mm to (39.4, 46.5)
- moved R6 2.06 mm to (36.7, 39.0)
Connections:
- new net N$99: D1.A, IC1.3, J3.2
- net 0V: now also J3.1; no longer D1.A, IC1.2
- net N$1: now also IC1.2; no longer IC1.3
Routing:
- net L_G: track 19.2 -> 56.7 mm
- net N$99: track 0.00 -> 23.1 mm
- net N$6: track 56.8 -> 39.5 mm
- net N$7: track 16.0 -> 25.7 mm
- net N$13: track 29.7 -> 38.3 mm
- net 4.5V: track 22.6 -> 27.2 mm
- net 12V: track 60.1 -> 62.8 mm
- net N$3: track 4.76 -> 6.36 mm
- net N$1: track 55.9 -> 54.3 mm
- net N$8: track 6.70 -> 5.44 mm
- net N$12: track 5.44 -> 4.39 mm

Commit message: included figure of the adc board
Parts:
- removed J3: (no value), con-amp:10X02MTA
- added C1: 10 pf, capacitor-wima:C5B2.5
- Q1, Q2, Q3: value (none) -> NTD5867NL
Connections:
- removed net N$99: D1.A, IC1.3, J3.2
- net 0V: now also D1.A, IC1.3; no longer J3.1
- net N$1: now also C1.1
- net N$7: now also C1.2
Routing:
- net N$99: track 23.1 -> 0.00 mm
- net 0V: track 0.00 -> 22.6 mm
Changed lines of the file:
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@@
 <element name="R3" library="rcl" package="0207/10" value="1.2K" x="26.322" y="58.741" rot="R270"/>
 <element name="LED_RED" library="adafruit" package="LED5MM" value="" x="48.0765" y="49.59" rot="R270"/>
-<element name="Q1" library="adafruit" package="TO220V" value="" x="72.77" y="51.1" rot="R270"/>
+<element name="Q1" library="adafruit" package="TO220V" value="NTD5867NL" x="72.77" y="51.1" rot="R270"/>
 <element name="R5" library="rcl" package="0207/10" value="200" x="39.371" y="46.4515" rot="R225"/>
 <element name="LED_GREEN" library="adafruit" package="LED5MM" value="" x="43.004" y="43.2555"/>
-<element name="Q2" library="adafruit" package="TO220V" value="" x="67.18" y="50.85" rot="R270"/>
+<element name="Q2" library="adafruit" package="TO220V" value="NTD5867NL" x="67.18" y="50.85" rot="R270"/>
 <element name="R6" library="rcl" package="0207/10" value="160" x="36.702" y="39.0025" rot="R180"/>
 <element name="LED_BLUE" library="adafruit" package="LED5MM" value="" x="53.9705" y="43.2555" rot="R180"/>
-<element name="Q3" library="adafruit" package="TO220V" value="" x="61.3" y="51.1" rot="R270"/>
+<element name="Q3" library="adafruit" package="TO220V" value="NTD5867NL" x="61.3" y="51.1" rot="R270"/>
 <element name="R7" library="rcl" package="0207/10" value="160" x="59.24" y="39.45" rot="R270"/>
 <element name="J1" library="con-amp" package="10X08MTA" value="" x="55.84" y="68.327"/>
@@
 <element name="R10" library="rcl" package="0207/10" value="12K" x="64.75" y="64" rot="R180"/>
 <element name="R2" library="rcl" package="0207/10" value="7.5K" x="36.8145" y="33.985" rot="R180"/>
-<element name="J3" library="con-amp" package="10X02MTA" value="" x="47.9425" y="37.719" rot="R270"/>
+<element name="C1" library="capacitor-wima" package="C5B2.5" value="10 pf" x="4.318" y="-3.2385"/>
 </elements>
 <signals>
@@
 <wire x1="34.29" y1="54.61" x2="34.29" y2="52.07" width="0.4572" layer="1"/>
 <wire x1="36.83" y1="49.53" x2="37.0721" y2="48.967896875" width="0.4572" layer="1"/>
+<contactref element="C1" pad="2"/>
+<wire x1="6.858" y1="-3.2385" x2="31.92" y2="42.8" width="0" layer="19" extent="1-1"/>
 </signal>
 <signal name="12V">
@@
 <contactref element="R4" pad="2"/>
 <contactref element="IC1" pad="4"/>
-<contactref element="J3" pad="1"/>
+<contactref element="D1" pad="A"/>
+<contactref element="IC1" pad="3"/>
+<wire x1="48.26" y1="39.37" x2="48.26" y2="41.91" width="0.4572" layer="1"/>
+<wire x1="34.29" y1="48.26" x2="31.75" y2="48.26" width="0.4572" layer="1"/>
+<wire x1="36.83" y1="45.72" x2="34.29" y2="48.26" width="0.4572" layer="1"/>
+<wire x1="44.45" y1="45.72" x2="36.83" y2="45.72" width="0.4572" layer="1"/>
+<wire x1="48.26" y1="41.91" x2="44.45" y2="45.72" width="0.4572" layer="1"/>
+<wire x1="31.75" y1="48.26" x2="31.92" y2="47.88" width="0.4572" layer="1"/>
+<wire x1="48.26" y1="41.91" x2="47.89" y2="42.18" width="0.4572" layer="1"/>
+<wire x1="80.08" y1="58" x2="76.58" y2="60.75" width="0" layer="19" extent="1-1"/>
+<wire x1="69.83" y1="64" x2="76.58" y2="60.75" width="0" layer="19" extent="1-1"/>
+<wire x1="70.23" y1="48.56" x2="80.08" y2="58" width="0" layer="19" extent="1-1"/>
 <wire x1="64.64" y1="48.31" x2="70.23" y2="48.56" width="0" layer="19" extent="1-1"/>
 <wire x1="58.76" y1="48.56" x2="64.64" y2="48.31" width="0" layer="19" extent="1-1"/>
+<wire x1="48.26" y1="41.91" x2="58.76" y2="48.56" width="0" layer="19" extent="1-1"/>
+<wire x1="31.92" y1="50.42" x2="31.75" y2="48.26" width="0" layer="19" extent="1-1"/>
+<wire x1="23.305" y1="53.605" x2="31.92" y2="50.42" width="0" layer="19" extent="1-1"/>
+<wire x1="70.971" y1="34.4905" x2="70.23" y2="48.56" width="0" layer="19" extent="1-1"/>
 <wire x1="54.86" y1="62.85" x2="58.76" y2="48.56" width="0" layer="19" extent="1-1"/>
-<wire x1="31.92" y1="50.42" x2="23.305" y2="53.605" width="0" layer="19" extent="1-1"/>
+<wire x1="42.16" y1="62.85" x2="54.86" y2="62.85" width="0" layer="19" extent="1-1"/>
 </signal>
 <signal name="CLK">
@@
 <wire x1="46.99" y1="44.45" x2="47.89" y2="44.72" width="0.4572" layer="1"/>
 <wire x1="31.75" y1="45.72" x2="31.92" y2="45.34" width="0.4572" layer="1"/>
+<contactref element="C1" pad="1"/>
+<wire x1="1.778" y1="-3.2385" x2="30.48" y2="40.64" width="0" layer="19" extent="1-1"/>
 </signal>
 <signal name="3.3V">
@@
 <wire x1="26.67" y1="53.34" x2="26.322" y2="53.661" width="0.4572" layer="1"/>
 </signal>
-<signal name="N$99">
-<contactref element="D1" pad="A"/>
-<contactref element="J3" pad="2"/>
-<contactref element="IC1" pad="3"/>
-<wire x1="48.26" y1="39.37" x2="48.26" y2="41.91" width="0.4572" layer="1"/>
-<wire x1="48.26" y1="39.37" x2="47.9425" y2="38.989" width="0.4572" layer="1"/>
-<wire x1="34.29" y1="48.26" x2="31.75" y2="48.26" width="0.4572" layer="1"/>
-<wire x1="36.83" y1="45.72" x2="34.29" y2="48.26" width="0.4572" layer="1"/>
-<wire x1="44.45" y1="45.72" x2="36.83" y2="45.72" width="0.4572" layer="1"/>
-<wire x1="48.26" y1="41.91" x2="44.45" y2="45.72" width="0.4572" layer="1"/>
-<wire x1="31.75" y1="48.26" x2="31.92" y2="47.88" width="0.4572" layer="1"/>
-<wire x1="48.26" y1="41.91" x2="47.89" y2="42.18" width="0.4572" layer="1"/>
-</signal>
 </signals>

Commit message: eagle files
Parts:
- IC1: value LM358N -> LM2904
Changed lines of the file:
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@@
 <element name="J1" library="con-amp" package="10X08MTA" value="" x="55.84" y="68.327"/>
 <element name="J2" library="my_lbr" package="10X03MTA" value="" x="70.971" y="37.0305" rot="R270"/>
-<element name="IC1" library="linear" package="DIL08" value="LM358N" x="28.11" y="46.61" rot="R90"/>
+<element name="IC1" library="linear" package="DIL08" value="LM2904" x="28.11" y="46.61" rot="R90"/>
 <element name="R8" library="rcl" package="0207/10" value="12K" x="75" y="58"/>
 <element name="R9" library="rcl" package="0207/10" value="12K" x="71.5" y="60.75"/>
