File: emb/rotating_clock/pcb/board.brd (EAGLE design)
At the start: 104.6 x 80.3 mm, 44 parts, among them IC1 CAT4016, IC2 CAT4016

Commit message: added slip ring board
Parts:
- removed PAD1: LATCH, wirepad:3,17/1,3
- removed PAD2: SIN, wirepad:3,17/1,3
- removed PAD3: CLK, wirepad:3,17/1,3
- removed PAD4: GND, wirepad:3,17/1,3
- removed PAD5: 5V, wirepad:3,17/1,3
- added U$1: SLIP-RING-INVERSE, slip_ring:SLIP-RING-INVERSE
Connections:
- net 5V: now also U$1.3V3; no longer PAD5.1
- net CLK: now also U$1.CLK; no longer PAD3.1
- net GND: now also U$1.GND; no longer PAD4.1
- net LATCH: now also U$1.SIG2.1, U$1.SIG2.2; no longer PAD1.1
- net SIN: now also U$1.SIG1.1, U$1.SIG1.2; no longer PAD2.1
Routing:
- net SIN: track 29.6 -> 102.1 mm
- net GND: track 266.3 -> 317.6 mm
- net LATCH: track 96.2 -> 54.3 mm, vias 1 -> 0
- net 5V: track 82.7 -> 57.7 mm
- net CLK: track 84.7 -> 101.0 mm
Other:
- board text added: "LED board"
