File: emb/rotating_clock/pcb/top_board/board.brd (EAGLE design)
At the start: 104.6 x 80 mm, 39 parts, among them IC1 CAT4016, IC2 CAT4016

Commit message: Updated board
Parts:
- moved C2 3.57 mm to (6.35, 48.3)
Routing:
- net N$39: track 203.6 -> 181.1 mm
- net 5V: track 104.6 -> 110.5 mm, vias 2 -> 3
- added copper zone on layer 16, net N$36
- added copper zone on layer 1, net N$38
- added copper zone on layer 1, net N$39
- added copper zone on layer 16, net N$39
Changed lines of the file:
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@@
 <grid distance="0.01" unitdist="inch" unit="inch" style="lines" multiple="1" display="no" altdistance="0.025" altunitdist="inch" altunit="inch"/>
 <layers>
-<layer number="1" name="Top" color="4" fill="1" visible="yes" active="yes"/>
+<layer number="1" name="Top" color="4" fill="1" visible="no" active="yes"/>
 <layer number="16" name="Bottom" color="1" fill="1" visible="yes" active="yes"/>
 <layer number="17" name="Pads" color="2" fill="1" visible="yes" active="yes"/>
 <layer number="18" name="Vias" color="2" fill="1" visible="yes" active="yes"/>
-<layer number="19" name="Unrouted" color="6" fill="1" visible="yes" active="yes"/>
-<layer number="20" name="Dimension" color="15" fill="1" visible="yes" active="yes"/>
-<layer number="21" name="tPlace" color="7" fill="1" visible="yes" active="yes"/>
-<layer number="22" name="bPlace" color="7" fill="1" visible="yes" active="yes"/>
-<layer number="23" name="tOrigins" color="15" fill="1" visible="yes" active="yes"/>
-<layer number="24" name="bOrigins" color="15" fill="1" visible="yes" active="yes"/>
-<layer number="25" name="tNames" color="7" fill="1" visible="yes" active="yes"/>
-<layer number="26" name="bNames" color="7" fill="1" visible="yes" active="yes"/>
-<layer number="27" name="tValues" color="7" fill="1" visible="yes" active="yes"/>
-<layer number="28" name="bValues" color="7" fill="1" visible="yes" active="yes"/>
+<layer number="19" name="Unrouted" color="6" fill="1" visible="no" active="yes"/>
+<layer number="20" name="Dimension" color="15" fill="1" visible="no" active="yes"/>
+<layer number="21" name="tPlace" color="7" fill="1" visible="no" active="yes"/>
+<layer number="22" name="bPlace" color="7" fill="1" visible="no" active="yes"/>
+<layer number="23" name="tOrigins" color="15" fill="1" visible="no" active="yes"/>
+<layer number="24" name="bOrigins" color="15" fill="1" visible="no" active="yes"/>
+<layer number="25" name="tNames" color="7" fill="1" visible="no" active="yes"/>
+<layer number="26" name="bNames" color="7" fill="1" visible="no" active="yes"/>
+<layer number="27" name="tValues" color="7" fill="1" visible="no" active="yes"/>
+<layer number="28" name="bValues" color="7" fill="1" visible="no" active="yes"/>
 <layer number="29" name="tStop" color="7" fill="3" visible="no" active="yes"/>
 <layer number="30" name="bStop" color="7" fill="6" visible="no" active="yes"/>
@@
 <layer number="37" name="tTest" color="7" fill="1" visible="no" active="yes"/>
 <layer number="38" name="bTest" color="7" fill="1" visible="no" active="yes"/>
-<layer number="39" name="tKeepout" color="4" fill="11" visible="yes" active="yes"/>
-<layer number="40" name="bKeepout" color="1" fill="11" visible="yes" active="yes"/>
-<layer number="41" name="tRestrict" color="4" fill="10" visible="yes" active="yes"/>
-<layer number="42" name="bRestrict" color="1" fill="10" visible="yes" active="yes"/>
-<layer number="43" name="vRestrict" color="2" fill="10" visible="yes" active="yes"/>
+<layer number="39" name="tKeepout" color="4" fill="11" visible="no" active="yes"/>
+<layer number="40" name="bKeepout" color="1" fill="11" visible="no" active="yes"/>
+<layer number="41" name="tRestrict" color="4" fill="10" visible="no" active="yes"/>
+<layer number="42" name="bRestrict" color="1" fill="10" visible="no" active="yes"/>
+<layer number="43" name="vRestrict" color="2" fill="10" visible="no" active="yes"/>
 <layer number="44" name="Drills" color="7" fill="1" visible="no" active="yes"/>
 <layer number="45" name="Holes" color="7" fill="1" visible="no" active="yes"/>
 <layer number="46" name="Milling" color="3" fill="1" visible="no" active="yes"/>
 <layer number="47" name="Measures" color="7" fill="1" visible="no" active="yes"/>
-<layer number="48" name="Document" color="7" fill="1" visible="yes" active="yes"/>
-<layer number="49" name="Reference" color="7" fill="1" visible="yes" active="yes"/>
-<layer number="51" name="tDocu" color="7" fill="1" visible="yes" active="yes"/>
-<layer number="52" name="bDocu" color="7" fill="1" visible="yes" active="yes"/>
+<layer number="48" name="Document" color="7" fill="1" visible="no" active="yes"/>
+<layer number="49" name="Reference" color="7" fill="1" visible="no" active="yes"/>
+<layer number="51" name="tDocu" color="7" fill="1" visible="no" active="yes"/>
+<layer number="52" name="bDocu" color="7" fill="1" visible="no" active="yes"/>
 <layer number="90" name="Modules" color="5" fill="1" visible="no" active="no"/>
 <layer number="91" name="Nets" color="2" fill="1" visible="no" active="no"/>
@@
 <wire x1="0" y1="-0.254" x2="104.572" y2="-0.254" width="0" layer="20"/>
 <wire x1="104.572" y1="-0.254" x2="104.572" y2="79.746" width="0" layer="20"/>
-<wire x1="104.572" y1="79.746" x2="0" y2="79.746" width="0" layer="20"/>
 <wire x1="0" y1="79.746" x2="0" y2="-0.254" width="0" layer="20"/>
 <text x="59.182" y="32.004" size="1.778" layer="16" rot="MR0">LED board</text>
@@
 <element name="LED31" library="led" package="CHIPLED-0603-TTW" value="" x="96.52" y="39.37" rot="R180"/>
 <element name="LED32" library="led" package="CHIPLED-0603-TTW" value="" x="99.06" y="39.37" rot="R180"/>
-<element name="C2" library="rcl" package="E5-8,5" value="220 µF" x="2.794" y="48.006" rot="R180"/>
+<element name="C2" library="rcl" package="E5-8,5" value="220 µF" x="6.35" y="48.26" rot="R180"/>
 <element name="C1" library="rcl" package="E5-8,5" value="15 pF" x="95.758" y="53.848"/>
 <element name="U$1" library="slip_ring" package="SLIP-RING-INVERSE" value="SLIP-RING-INVERSE" x="18.288" y="38.862" rot="R210"/>
@@
 <wire x1="39.37" y1="55.245" x2="40.64" y2="56.515" width="0.6096" layer="16"/>
 <wire x1="12.7" y1="55.245" x2="39.37" y2="55.245" width="0.6096" layer="16"/>
-<wire x1="5.715" y1="48.26" x2="12.7" y2="55.245" width="0.6096" layer="16"/>
 <wire x1="43.815" y1="56.515" x2="44.224" y2="56.261" width="0.6096" layer="1"/>
-<wire x1="5.715" y1="48.26" x2="5.334" y2="48.006" width="0.6096" layer="16"/>
 <wire x1="82.55" y1="56.515" x2="84.455" y2="56.515" width="0.6096" layer="1"/>
 <wire x1="81.28" y1="55.245" x2="82.55" y2="56.515" width="0.6096" layer="16"/>
 <wire x1="39.37" y1="55.245" x2="81.28" y2="55.245" width="0.6096" layer="16"/>
 <wire x1="84.455" y1="56.515" x2="84.61" y2="56.769" width="0.6096" layer="1"/>
-<wire x1="6.35" y1="47.625" x2="15.875" y2="38.1" width="0.6096" layer="16"/>
-<wire x1="5.715" y1="47.625" x2="6.35" y2="47.625" width="0.6096" layer="16"/>
-<wire x1="15.875" y1="38.1" x2="16.08829375" y2="37.592" width="0.6096" layer="16"/>
-<wire x1="5.715" y1="47.625" x2="5.334" y2="48.006" width="0.6096" layer="16"/>
 <via x="40.64" y="56.515" extent="1-16" drill="0.6096"/>
 <via x="82.55" y="56.515" extent="1-16" drill="0.6096"/>
+<wire x1="16.08829375" y1="37.592" x2="16.08829375" y2="36.66229375" width="0.4064" layer="1"/>
+<wire x1="16.08829375" y1="36.66229375" x2="12.7" y2="33.274" width="0.4064" layer="1"/>
+<wire x1="12.7" y1="33.274" x2="11.938" y2="33.274" width="0.4064" layer="1"/>
+<wire x1="11.938" y1="33.274" x2="9.144" y2="36.068" width="0.4064" layer="1"/>
+<wire x1="9.144" y1="36.068" x2="9.144" y2="48.006" width="0.4064" layer="1"/>
+<wire x1="9.144" y1="48.006" x2="8.89" y2="48.26" width="0.4064" layer="1"/>
+<wire x1="8.89" y1="48.26" x2="8.89" y2="51.562" width="0.4064" layer="1"/>
+<wire x1="8.89" y1="51.562" x2="10.414" y2="53.086" width="0.4064" layer="1"/>
+<via x="10.414" y="53.086" extent="1-16" drill="0.6"/>
+<wire x1="10.414" y1="53.086" x2="10.541" y2="53.086" width="0.4064" layer="16"/>
+<wire x1="10.541" y1="53.086" x2="12.7" y2="55.245" width="0.4064" layer="16"/>
 </signal>
 <signal name="N$1">
@@
 <wire x1="39.37" y1="56.515" x2="39.37" y2="58.42" width="0.6096" layer="1"/>
 <wire x1="57.785" y1="57.15" x2="58.166" y2="56.896" width="0.6096" layer="1"/>
-<wire x1="0.254" y1="48.006" x2="0.254" y2="45.212" width="0.6096" layer="1"/>
-<wire x1="0.254" y1="45.212" x2="14.224" y2="31.242" width="0.6096" layer="1"/>
 <wire x1="14.224" y1="31.242" x2="17.95438125" y2="31.242" width="0.6096" layer="1"/>
 <wire x1="17.95438125" y1="31.242" x2="20.955" y2="34.24261875" width="0.6096" layer="1"/>
+<polygon width="0.4064" layer="1">
+<vertex x="103.378" y="59.182"/>
+<vertex x="103.378" y="18.288"/>
+<vertex x="-103.124" y="18.288"/>
+<vertex x="-103.124" y="59.182"/>
+</polygon>
+<polygon width="0.4064" layer="16">
+<vertex x="103.378" y="59.182"/>
+<vertex x="-103.124" y="59.182"/>
+<vertex x="-103.124" y="18.288"/>
+<vertex x="103.378" y="18.288"/>
+</polygon>
+</signal>
+<signal name="N$35">
+<via x="10.414" y="53.086" extent="1-16" drill="0.6"/>
+</signal>
+<signal name="N$36">
+<polygon width="0.4064" layer="16">
+<vertex x="1.016" y="59.182"/>
+<vertex x="-103.124" y="59.182"/>
+<vertex x="-103.124" y="18.288"/>
+<vertex x="1.016" y="18.288"/>
+</polygon>
+</signal>
+<signal name="N$37">
+<via x="18.288" y="38.862" extent="1-16" drill="0.6"/>
+</signal>
+<signal name="N$38">
+<polygon width="0.4064" layer="1">
+<vertex x="-103.124" y="59.182"/>
+<vertex x="-1.016" y="59.182"/>
+<vertex x="-1.016" y="18.288"/>
+<vertex x="-103.124" y="18.288"/>
+</polygon>
 </signal>
 </signals>
